Commit message: 5th practical session

File: src/my_r2d2/urdf/final.xacro (robot description, xacro)
@@ -417,3 +417,10 @@
     <origin xyz="0 0 0.45"/>
   </joint>
+//-------------------------------------------------------------------
+  <link name="eye" type="fixed"/>
+  <joint name="lense_to_eye" type="fixed">
+     <parent link="lense"/>
+     <child link="eye"/>
+     <origin xyz="0.5 0 0" rpy="0 1.571 1.571"/> // 4.713
+  </joint>
 </robot>
