Commit message: Adding final changes form third practical

File: src/my_r2d2/urdf/final.urdf (robot description, URDF)
Before this commit: robot final_robot, 16 links, 15 joints
Links:
- added link lense, mass 1; visual cylinder length=0.02 radius=0.0266666666667
Joints:
- added joint to_lens: type fixed, parent box, child lense

File: src/my_r2d2/urdf/final.xacro (robot description, xacro)
@@ -1,12 +1,12 @@
 <?xml version="1.0"?>
 <robot xmlns:xacro="http://www.ros.org/wiki/xacro" name="final_robot">
-<material name="blue">
-    <color rgba="0 0 0.8 1"/>
+  <material name="blue">
+    <color rgba="0 0 0.8 2"/>
   </material>
   <material name="black">
-    <color rgba="0 0 0 1"/>
+    <color rgba="0 0 0 2"/>
   </material>
   <material name="white">
-    <color rgba="1 1 1 1"/>
+    <color rgba="1 1 1 2"/>
   </material>
   <link name="base_link">
@@ -361,12 +361,16 @@
   </joint>
 //-----------------------------------------------
-  <xacro:property name="box_param" value="0.8" />
-  <xacro:macro name="box_origin">
-    <origin xyz="-0.04 0 0"/>
+  <xacro:property name="box_param" value="0.08" />
+  <xacro:macro name="lens_geometry">
+    <geometry>
+      <cylinder radius="${box_param/3}" length="${box_param/4}"/>
+    </geometry>
   </xacro:macro>
-  <xacro:macro name="lens_visual">
-    <visual>
-      <geometry>
-        <cylinder
+  <xacro:macro name="box_inertial">
+    <inertial>
+      <mass value="1"/>
+      <inertia ixx="1.0" ixy="0.0" ixz="0.0" iyy="1.0" iyz="0.0" izz="1.0"/>
+    </inertial>
+  </xacro:macro>
   <link name="box">
     <visual>
@@ -375,5 +379,5 @@
       </geometry>
       <material name="blue"/>
-      <xacro:box_origin/>
+      <origin xyz = "-0.04 0 0"/>
     </visual>
     <collision>
@@ -382,8 +386,5 @@
       </geometry>
     </collision>
-    <inertial>
-      <mass value="1"/>
-      <inertia ixx="1.0" ixy="0.0" ixz="0.0" iyy="1.0" iyz="0.0" izz="1.0"/>
-    </inertial>
+      <xacro:box_inertial/>
   </link>
   <joint name="tobox" type="fixed">
@@ -394,5 +395,16 @@
   <link name="lense">
     <visual>
-      <geometry>
-        <cylinder
+      <xacro:lens_geometry/>
+      <origin rpy="0 1.571 0" xyz="-0.009 0 0"/>
+      <material name="black"/>
+    </visual>
+    <collison>
+      <xacro:lens_geometry/>
+    </collison>
+    <xacro:box_inertial/>
+  </link>
+//  <joint name="to_lens" type="fixed">
+//    <parent link="box"/>
+//    <child link="lense"/>
+//  </joint>
 </robot>

Commit message: Things related to third practical and fourth practical

File: src/my_r2d2/urdf/final.urdf (robot description, URDF)
Before this commit: robot final_robot, 17 links, 16 joints
Links:
- added link base_footprint
Joints:
- added joint base_footprint_to_base_link: type fixed, parent base_footprint, child base_link, origin xyz=0 0 0.45
- joint to_lens: origin (none) -> xyz=-0.009 0 0

File: src/my_r2d2/urdf/final.xacro (robot description, xacro)
@@ -396,5 +396,5 @@
     <visual>
       <xacro:lens_geometry/>
-      <origin rpy="0 1.571 0" xyz="-0.009 0 0"/>
+      <origin rpy="0 1.571 0"/>
       <material name="black"/>
     </visual>
@@ -404,7 +404,16 @@
     <xacro:box_inertial/>
   </link>
-//  <joint name="to_lens" type="fixed">
-//    <parent link="box"/>
-//    <child link="lense"/>
-//  </joint>
+  <joint name="to_lens" type="fixed">
+    <origin xyz="-0.009 0 0"/>
+    <parent link="box"/>
+    <child link="lense"/>
+  </joint>
+//------------------------------------------------------------------
+  <link name="base_footprint">
+  </link>
+  <joint name="base_footprint_to_base_link" type="fixed">
+    <parent link="base_footprint"/>
+    <child link="base_link"/>
+    <origin xyz="0 0 0.45"/>
+  </joint>
 </robot>

Commit message: Finishing touches on 5th practical

File: src/my_r2d2/urdf/final.urdf (robot description, URDF)
Before this commit: robot final_robot, 19 links, 18 joints
Joints:
- joint lense_to_eye: origin xyz=0.5 0 0 rpy=0 1.571 1.571 -> xyz=-0.009 0 0 rpy=1.571 3.142 1.571

File: src/my_r2d2/urdf/final.xacro (robot description, xacro)
@@ -422,5 +422,5 @@
      <parent link="lense"/>
      <child link="eye"/>
-     <origin xyz="0.5 0 0" rpy="0 1.571 1.571"/> // 4.713
+     <origin xyz="-0.009 0 0" rpy="1.571 3.142 1.571"/> // 4.713
   </joint>
 </robot>
