Commit message: Finishing the last practical

File: src/dual_manipulator_support/urdf/dual_man_2.xacro (robot description, xacro)
@@ -15,6 +15,7 @@
 	<xacro:include filename="$(find motoman_sia5d_support)/urdf/sia5d_macro.xacro"/>
 	<xacro:motoman_sia5d prefix="1"/>
-	<xacro:include filename="$(find motoman_sia5d_support)/urdf/sia5d_macro.xacro"/>
-	<xacro:motoman_sia5d prefix="2"/>
+<!--ur5 part begins-->
+	<xacro:include filename="$(find ur_description)/urdf/ur5_robot.urdf.xacro"/>
+<!--ur5 part ends -->
 <joint name="base_to_robot_1" type="fixed">
 	<parent link="base_link"/>
@@ -24,5 +25,5 @@
 <joint name="base_to_robot_2" type="fixed">
 	<parent link="base_link"/>
-	<child link="2base_link"/>
+	<child link="_base_link"/>
 	<origin xyz="0 -0.5 0.1"/>
 </joint>
