Commit message: Final touches to the last practical

File: src/dual_manipulator_support/urdf/dual_man_2.urdf (robot description, URDF)
Before this commit: robot dual_manipulator, 21 links, 20 joints
Links:
- added link world
Joints:
- removed joint _base_link-base_fixed_joint
- added joint base_link-base_fixed_joint: type fixed, parent _base_link, child base, origin xyz=0 0 0 rpy=0 0 -3.14159265359
- added joint world_joint: type fixed, parent world, child base_link, origin xyz=0.0 0.0 0.0 rpy=0.0 0.0 0.0

File: src/dual_manipulator_support/urdf/dual_man_2.xacro (robot description, xacro)
@@ -16,5 +16,5 @@
 	<xacro:motoman_sia5d prefix="1"/>
 <!--ur5 part begins-->
-	<xacro:include filename="$(find ur_description)/urdf/ur5_robot.urdf.xacro"/>
+	<xacro:include filename="/home/roberts/roberts-rtech/src/dual_manipulator_support/ur_description_edit/urdf/ur5_robot.urdf.xacro"/>
 <!--ur5 part ends -->
 <joint name="base_to_robot_1" type="fixed">
